Commit message: エラー修正、アームが一切うごかない

File: install/mizuki_arm_short/share/mizuki_arm_short/urdf/arm_v20(2).SLDASM.urdf (robot description, URDF)
Before this commit: robot arm_v20(2).SLDASM, 7 links, 6 joints
Links:
- link base_link: mass 0.727427477022971 -> None

File: install/moveit_config/share/moveit_config/config/arm_v20(2).SLDASM.ros2_control.xacro (robot description, xacro)
@@ -2,5 +2,5 @@
 <robot xmlns:xacro="http://www.ros.org/wiki/xacro">
     <xacro:macro name="arm_v20_2_SLDASM_ros2_control" params="name initial_positions_file">
-        <xacro:property name="initial_positions" value="${load_yaml(initial_positions_file)['initial_positions']}"/>
+        <xacro:property name="initial_positions" value="${xacro.load_yaml(initial_positions_file)['initial_positions']}"/>
         <ros2_control name="${name}" type="system">
             <hardware>
