Commit message: urdf表示された

File: install/arm_v20_description/share/arm_v20_description/urdf/arm_v20.xacro (robot description, xacro)
@@ -1,6 +1,6 @@
 <?xml version="1.0" ?>
-<robot name="arm_v20(2)" xmlns:xacro="http://www.ros.org/wiki/xacro">
-<xacro:include filename="$(find arm_v20(2)_description)/urdf/materials.xacro" />
-<xacro:include filename="$(find arm_v20(2)_description)/urdf/arm_v20(2).trans" />
+<robot name="arm_v20" xmlns:xacro="http://www.ros.org/wiki/xacro">
+<xacro:include filename="$(find arm_v20_description)/urdf/materials.xacro" />
+<xacro:include filename="$(find arm_v20_description)/urdf/arm_v20.trans" />
 <link name="base_link">
   <inertial>
@@ -12,5 +12,5 @@
     <origin xyz="0 0 0" rpy="0 0 0"/>
     <geometry>
-      <mesh filename="package://arm_v20(2)_description/meshes/base_link.stl" scale="0.001 0.001 0.001"/>
+      <mesh filename="package://arm_v20_description/meshes/base_link.stl" scale="0.001 0.001 0.001"/>
     </geometry>
     <material name="silver_default"/>
@@ -19,5 +19,5 @@
     <origin xyz="0 0 0" rpy="0 0 0"/>
     <geometry>
-      <mesh filename="package://arm_v20(2)_description/meshes/base_link.stl" scale="0.001 0.001 0.001"/>
+      <mesh filename="package://arm_v20_description/meshes/base_link.stl" scale="0.001 0.001 0.001"/>
     </geometry>
   </collision>
@@ -32,5 +32,5 @@
     <origin xyz="-0.0 0.0 -0.0525" rpy="0 0 0"/>
     <geometry>
-      <mesh filename="package://arm_v20(2)_description/meshes/link1_1.stl" scale="0.001 0.001 0.001"/>
+      <mesh filename="package://arm_v20_description/meshes/link1_1.stl" scale="0.001 0.001 0.001"/>
     </geometry>
     <material name="opaque202209238"/>
@@ -39,5 +39,5 @@
     <origin xyz="-0.0 0.0 -0.0525" rpy="0 0 0"/>
     <geometry>
-      <mesh filename="package://arm_v20(2)_description/meshes/link1_1.stl" scale="0.001 0.001 0.001"/>
+      <mesh filename="package://arm_v20_description/meshes/link1_1.stl" scale="0.001 0.001 0.001"/>
     </geometry>
   </collision>
@@ -52,5 +52,5 @@
     <origin xyz="-2.1e-05 -0.024521 -0.123563" rpy="0 0 0"/>
     <geometry>
-      <mesh filename="package://arm_v20(2)_description/meshes/link2_1.stl" scale="0.001 0.001 0.001"/>
+      <mesh filename="package://arm_v20_description/meshes/link2_1.stl" scale="0.001 0.001 0.001"/>
     </geometry>
     <material name="opaque202209238"/>
@@ -59,5 +59,5 @@
     <origin xyz="-2.1e-05 -0.024521 -0.123563" rpy="0 0 0"/>
     <geometry>
-      <mesh filename="package://arm_v20(2)_description/meshes/link2_1.stl" scale="0.001 0.001 0.001"/>
+      <mesh filename="package://arm_v20_description/meshes/link2_1.stl" scale="0.001 0.001 0.001"/>
     </geometry>
   </collision>
@@ -72,5 +72,5 @@
     <origin xyz="-0.034771 -0.012321 -0.265313" rpy="0 0 0"/>
     <geometry>
-      <mesh filename="package://arm_v20(2)_description/meshes/link3_1.stl" scale="0.001 0.001 0.001"/>
+      <mesh filename="package://arm_v20_description/meshes/link3_1.stl" scale="0.001 0.001 0.001"/>
     </geometry>
     <material name="steel_satin"/>
@@ -79,5 +79,5 @@
     <origin xyz="-0.034771 -0.012321 -0.265313" rpy="0 0 0"/>
     <geometry>
-      <mesh filename="package://arm_v20(2)_description/meshes/link3_1.stl" scale="0.001 0.001 0.001"/>
+      <mesh filename="package://arm_v20_description/meshes/link3_1.stl" scale="0.001 0.001 0.001"/>
     </geometry>
   </collision>
@@ -92,5 +92,5 @@
     <origin xyz="-0.170171 0.000179 -0.265313" rpy="0 0 0"/>
     <geometry>
-      <mesh filename="package://arm_v20(2)_description/meshes/link4_1.stl" scale="0.001 0.001 0.001"/>
+      <mesh filename="package://arm_v20_description/meshes/link4_1.stl" scale="0.001 0.001 0.001"/>
     </geometry>
     <material name="silver_default"/>
@@ -99,5 +99,5 @@
     <origin xyz="-0.170171 0.000179 -0.265313" rpy="0 0 0"/>
     <geometry>
-      <mesh filename="package://arm_v20(2)_description/meshes/link4_1.stl" scale="0.001 0.001 0.001"/>
+      <mesh filename="package://arm_v20_description/meshes/link4_1.stl" scale="0.001 0.001 0.001"/>
     </geometry>
   </collision>
@@ -112,5 +112,5 @@
     <origin xyz="-0.248771 0.019079 -0.265313" rpy="0 0 0"/>
     <geometry>
-      <mesh filename="package://arm_v20(2)_description/meshes/link5_1.stl" scale="0.001 0.001 0.001"/>
+      <mesh filename="package://arm_v20_description/meshes/link5_1.stl" scale="0.001 0.001 0.001"/>
     </geometry>
     <material name="silver_default"/>
@@ -119,5 +119,5 @@
     <origin xyz="-0.248771 0.019079 -0.265313" rpy="0 0 0"/>
     <geometry>
-      <mesh filename="package://arm_v20(2)_description/meshes/link5_1.stl" scale="0.001 0.001 0.001"/>
+      <mesh filename="package://arm_v20_description/meshes/link5_1.stl" scale="0.001 0.001 0.001"/>
     </geometry>
   </collision>
@@ -132,5 +132,5 @@
     <origin xyz="-0.313771 0.000179 -0.265313" rpy="0 0 0"/>
     <geometry>
-      <mesh filename="package://arm_v20(2)_description/meshes/endeffector_1.stl" scale="0.001 0.001 0.001"/>
+      <mesh filename="package://arm_v20_description/meshes/endeffector_1.stl" scale="0.001 0.001 0.001"/>
     </geometry>
     <material name="silver_default"/>
@@ -139,5 +139,5 @@
     <origin xyz="-0.313771 0.000179 -0.265313" rpy="0 0 0"/>
     <geometry>
-      <mesh filename="package://arm_v20(2)_description/meshes/endeffector_1.stl" scale="0.001 0.001 0.001"/>
+      <mesh filename="package://arm_v20_description/meshes/endeffector_1.stl" scale="0.001 0.001 0.001"/>
     </geometry>
   </collision>

File: install/arm_v20_description/share/arm_v20_description/urdf/materials.xacro (robot description, xacro)
@@ -1,4 +1,4 @@
 <?xml version="1.0" ?>
-<robot name="arm_v20(2)" xmlns:xacro="http://www.ros.org/wiki/xacro" >
+<robot name="arm_v20" xmlns:xacro="http://www.ros.org/wiki/xacro" >
 <material name="silver_default">
   <color rgba="0.700 0.700 0.700 1.000"/>

Commit message: codex頑張れ後一歩

File: install/arm_v20_description/share/arm_v20_description/urdf/arm_v20.xacro (robot description, xacro)
@@ -143,5 +143,5 @@
   </collision>
 </link>
-<joint name="Revolute 1" type="continuous">
+<joint name="joint_1" type="continuous">
   <origin xyz="0.0 0.0 0.0525" rpy="0 0 0"/>
   <parent link="base_link"/>
@@ -149,5 +149,5 @@
   <axis xyz="-0.0 -0.0 1.0"/>
 </joint>
-<joint name="Revolute 2" type="revolute">
+<joint name="joint_2" type="revolute">
   <origin xyz="2.1e-05 0.024521 0.071063" rpy="0 0 0"/>
   <parent link="link1_1"/>
@@ -156,5 +156,5 @@
   <limit upper="1.570796" lower="-1.570796" effort="100" velocity="100"/>
 </joint>
-<joint name="Revolute 3" type="revolute">
+<joint name="joint_3" type="revolute">
   <origin xyz="0.03475 -0.0122 0.14175" rpy="0 0 0"/>
   <parent link="link2_1"/>
@@ -163,5 +163,5 @@
   <limit upper="1.570796" lower="-1.570796" effort="100" velocity="100"/>
 </joint>
-<joint name="Revolute 4" type="continuous">
+<joint name="joint_4" type="continuous">
   <origin xyz="0.1354 -0.0125 0.0" rpy="0 0 0"/>
   <parent link="link3_1"/>
@@ -169,5 +169,5 @@
   <axis xyz="1.0 -0.0 -0.0"/>
 </joint>
-<joint name="Revolute 5" type="revolute">
+<joint name="joint_5" type="revolute">
   <origin xyz="0.0786 -0.0189 0.0" rpy="0 0 0"/>
   <parent link="link4_1"/>
@@ -176,5 +176,5 @@
   <limit upper="1.570796" lower="-1.570796" effort="100" velocity="100"/>
 </joint>
-<joint name="Revolute 6" type="continuous">
+<joint name="joint_6" type="continuous">
   <origin xyz="0.065 0.0189 0.0" rpy="0 0 0"/>
   <parent link="link5_1"/>

File: install/moveit_config/share/moveit_config/config/arm_v20.ros2_control.xacro (robot description, xacro)
@@ -8,43 +8,43 @@
         <plugin>mock_components/GenericSystem</plugin>
       </hardware>
-      <joint name="Revolute 1">
+      <joint name="joint_1">
         <command_interface name="position"/>
         <state_interface name="position">
-          <param name="initial_value">${initial_positions['Revolute 1']}</param>
+          <param name="initial_value">${initial_positions['joint_1']}</param>
         </state_interface>
         <state_interface name="velocity"/>
       </joint>
-      <joint name="Revolute 2">
+      <joint name="joint_2">
         <command_interface name="position"/>
         <state_interface name="position">
-          <param name="initial_value">${initial_positions['Revolute 2']}</param>
+          <param name="initial_value">${initial_positions['joint_2']}</param>
         </state_interface>
         <state_interface name="velocity"/>
       </joint>
-      <joint name="Revolute 3">
+      <joint name="joint_3">
         <command_interface name="position"/>
         <state_interface name="position">
-          <param name="initial_value">${initial_positions['Revolute 3']}</param>
+          <param name="initial_value">${initial_positions['joint_3']}</param>
         </state_interface>
         <state_interface name="velocity"/>
       </joint>
-      <joint name="Revolute 4">
+      <joint name="joint_4">
         <command_interface name="position"/>
         <state_interface name="position">
-          <param name="initial_value">${initial_positions['Revolute 4']}</param>
+          <param name="initial_value">${initial_positions['joint_4']}</param>
         </state_interface>
         <state_interface name="velocity"/>
       </joint>
-      <joint name="Revolute 5">
+      <joint name="joint_5">
         <command_interface name="position"/>
         <state_interface name="position">
-          <param name="initial_value">${initial_positions['Revolute 5']}</param>
+          <param name="initial_value">${initial_positions['joint_5']}</param>
         </state_interface>
         <state_interface name="velocity"/>
       </joint>
-      <joint name="Revolute 6">
+      <joint name="joint_6">
         <command_interface name="position"/>
         <state_interface name="position">
-          <param name="initial_value">${initial_positions['Revolute 6']}</param>
+          <param name="initial_value">${initial_positions['joint_6']}</param>
         </state_interface>
         <state_interface name="velocity"/>

Commit message: SRDF等修正

File: install/arm_v20_description/share/arm_v20_description/urdf/arm_v20.xacro (robot description, xacro)
@@ -176,9 +176,10 @@
   <limit upper="1.570796" lower="-1.570796" effort="100" velocity="100"/>
 </joint>
-<joint name="joint_6" type="continuous">
+<joint name="joint_6" type="revolute">
   <origin xyz="0.065 0.0189 0.0" rpy="0 0 0"/>
   <parent link="link5_1"/>
   <child link="endeffector_1"/>
   <axis xyz="1.0 -0.0 -0.0"/>
+  <limit upper="3.14159265" lower="-3.14159265" effort="100" velocity="100"/>
 </joint>
 </robot>

File: install/moveit_config/share/moveit_config/config/arm_v20.ros2_control.xacro (robot description, xacro)
@@ -1,54 +1,54 @@
 <?xml version="1.0"?>
 <robot xmlns:xacro="http://www.ros.org/wiki/xacro">
-  <xacro:macro name="arm_v20_ros2_control" params="name initial_positions_file">
-    <xacro:property name="initial_positions" value="${xacro.load_yaml(initial_positions_file)['initial_positions']}"/>
-    <!-- シミュレーション向けに fake system を構成 -->
-    <ros2_control name="${name}" type="system">
-      <hardware>
-        <plugin>mock_components/GenericSystem</plugin>
-      </hardware>
-      <joint name="joint_1">
-        <command_interface name="position"/>
-        <state_interface name="position">
-          <param name="initial_value">${initial_positions['joint_1']}</param>
-        </state_interface>
-        <state_interface name="velocity"/>
-      </joint>
-      <joint name="joint_2">
-        <command_interface name="position"/>
-        <state_interface name="position">
-          <param name="initial_value">${initial_positions['joint_2']}</param>
-        </state_interface>
-        <state_interface name="velocity"/>
-      </joint>
-      <joint name="joint_3">
-        <command_interface name="position"/>
-        <state_interface name="position">
-          <param name="initial_value">${initial_positions['joint_3']}</param>
-        </state_interface>
-        <state_interface name="velocity"/>
-      </joint>
-      <joint name="joint_4">
-        <command_interface name="position"/>
-        <state_interface name="position">
-          <param name="initial_value">${initial_positions['joint_4']}</param>
-        </state_interface>
-        <state_interface name="velocity"/>
-      </joint>
-      <joint name="joint_5">
-        <command_interface name="position"/>
-        <state_interface name="position">
-          <param name="initial_value">${initial_positions['joint_5']}</param>
-        </state_interface>
-        <state_interface name="velocity"/>
-      </joint>
-      <joint name="joint_6">
-        <command_interface name="position"/>
-        <state_interface name="position">
-          <param name="initial_value">${initial_positions['joint_6']}</param>
-        </state_interface>
-        <state_interface name="velocity"/>
-      </joint>
-    </ros2_control>
-  </xacro:macro>
+    <xacro:macro name="arm_v20_ros2_control" params="name initial_positions_file">
+        <xacro:property name="initial_positions" value="${load_yaml(initial_positions_file)['initial_positions']}"/>
+        <ros2_control name="${name}" type="system">
+            <hardware>
+                <!-- By default, set up controllers for simulation. This won't work on real hardware -->
+                <plugin>mock_components/GenericSystem</plugin>
+            </hardware>
+            <joint name="Revolute 1">
+                <command_interface name="position"/>
+                <state_interface name="position">
+                  <param name="initial_value">${initial_positions['Revolute 1']}</param>
+                </state_interface>
+                <state_interface name="velocity"/>
+            </joint>
+            <joint name="Revolute 2">
+                <command_interface name="position"/>
+                <state_interface name="position">
+                  <param name="initial_value">${initial_positions['Revolute 2']}</param>
+                </state_interface>
+                <state_interface name="velocity"/>
+            </joint>
+            <joint name="Revolute 3">
+                <command_interface name="position"/>
+                <state_interface name="position">
+                  <param name="initial_value">${initial_positions['Revolute 3']}</param>
+                </state_interface>
+                <state_interface name="velocity"/>
+            </joint>
+            <joint name="Revolute 4">
+                <command_interface name="position"/>
+                <state_interface name="position">
+                  <param name="initial_value">${initial_positions['Revolute 4']}</param>
+                </state_interface>
+                <state_interface name="velocity"/>
+            </joint>
+            <joint name="Revolute 5">
+                <command_interface name="position"/>
+                <state_interface name="position">
+                  <param name="initial_value">${initial_positions['Revolute 5']}</param>
+                </state_interface>
+                <state_interface name="velocity"/>
+            </joint>
+            <joint name="Revolute 6">
+                <command_interface name="position"/>
+                <state_interface name="position">
+                  <param name="initial_value">${initial_positions['Revolute 6']}</param>
+                </state_interface>
+                <state_interface name="velocity"/>
+            </joint>
+        </ros2_control>
+    </xacro:macro>
 </robot>

File: install/moveit_config/share/moveit_config/config/arm_v20.urdf.xacro (robot description, xacro)
@@ -1,9 +1,9 @@
 <?xml version="1.0"?>
 <robot xmlns:xacro="http://www.ros.org/wiki/xacro" name="arm_v20">
-  <xacro:arg name="initial_positions_file" default="initial_positions.yaml"/>
-  <!-- 実機URDFの読み込み -->
-  <xacro:include filename="$(find arm_v20_description)/urdf/arm_v20.xacro"/>
-  <!-- ros2_control 用の設定を取り込み -->
-  <xacro:include filename="arm_v20.ros2_control.xacro"/>
-  <xacro:arm_v20_ros2_control name="FakeSystem" initial_positions_file="$(arg initial_positions_file)"/>
+    <xacro:arg name="initial_positions_file" default="initial_positions.yaml" />
+    <!-- Import arm_v20 urdf file -->
+    <xacro:include filename="$(find arm_v20_description)/urdf/arm_v20.urdf" />
+    <!-- Import control_xacro -->
+    <xacro:include filename="arm_v20.ros2_control.xacro" />
+    <xacro:arm_v20_ros2_control name="FakeSystem" initial_positions_file="$(arg initial_positions_file)"/>
 </robot>
