Commit message: odrive動かすコードを追加

File: install/a_r2_description/share/a_r2_description/urdf/a_r2.urdf (robot description, URDF)
Before this commit: robot a_r2, 6 links, 5 joints
Joints:
- joint Slider 4: limit lower=-0.6 upper=0.0 effort=100 velocity=100 -> lower=0.0 upper=0.6 effort=100 velocity=100

Commit message: 酒井a-mu#

File: install/a_r2_description/share/a_r2_description/urdf/a_r2.urdf (robot description, URDF)
Before this commit: robot a_r2, 6 links, 5 joints
Joints:
- joint Revolute 2: origin xyz=0.0285 0.102562 -0.065004 rpy=0 0 0 -> xyz=0.0285 0.102562 -0.065004 rpy=-0.436 0 0

Commit message: rthhethaのみにした、なぜかxyzでの指定がうまく行かないのでまた後で

File: install/a_r2_description/share/a_r2_description/urdf/a_r2.urdf (robot description, URDF)
Before this commit: robot a_r2, 6 links, 5 joints
Joints:
- joint Revolute 2: origin xyz=0.0285 0.102562 -0.065004 rpy=-0.436 0 0 -> xyz=0.0285 0.102562 -0.065004 rpy=-0.450 0 0
