Commit message: phiに対応

File: src/a_r2_description_v2/a_r2_description_v2/urdf/a_r2.urdf (robot description, URDF)
Before this commit: robot a_r2, 6 links, 5 joints
Links:
- added link link6_1, mass 1.4233723866284878; collision mesh filename=package://a_r2_description/meshes/link6_1.stl scale=0.001 0.001 0.001; visual mesh filename=package://a_r2_description/meshes/link6_1.stl scale=0.001 0.001 0.001
- link link5_1: mass 1.253566521763957 -> 0.007850000000000103
Joints:
- removed joint Slider 5
- added joint Revolute 5: type continuous, parent link4_1, child link5_1, origin xyz=0.0428 -0.020134 0.130121 rpy=0 0 0, axis 1.0 0.0 0.0
- added joint Slider 6: type prismatic, parent link5_1, child link6_1, origin xyz=0.01 0.0 0.0 rpy=0 0 0, axis 1.0 0.0 0.0, limit lower=0.0 upper=0.0 effort=100 velocity=100
- joint Revolute 2: origin xyz=0.0285 0.102562 -0.065004 rpy=-0.450 0 0 -> xyz=0.0285 0.102562 -0.065004 rpy=0 0 0
- joint Revolute 3: origin xyz=0.0 -0.188219 0.39771 rpy=0 0 0 -> xyz=0.0 0.009015 0.439907 rpy=0 0 0
- joint Slider 1: origin xyz=-0.279969 -1.870817 0.251713 rpy=0 0 0 -> xyz=-0.351158 -1.864523 0.253205 rpy=0 0 0
- joint Slider 4: axis -0.0 -0.440919 0.897547 -> -0.0 0.005889 0.999983; limit lower=0.0 upper=0.6 effort=100 velocity=100 -> lower=-0.6 upper=0.0 effort=100 velocity=100; origin xyz=0.0205 -0.170873 0.406231 rpy=0 0 0 -> xyz=0.0205 0.02834 0.439793 rpy=0 0 0

Commit message: rogilinkmsgを送信するようにした、path_commandのguiを追加した

File: src/a_r2_description_v2/a_r2_description_v2/urdf/a_r2.urdf (robot description, URDF)
Before this commit: robot a_r2, 7 links, 6 joints
Joints:
- joint Slider 4: limit lower=-0.6 upper=0.0 effort=100 velocity=100 -> lower=-0.6 upper=0.6 effort=100 velocity=100
- joint Slider 6: limit lower=0.0 upper=0.0 effort=100 velocity=100 -> lower=-0.1 upper=0.1 effort=100 velocity=100

File: src/a_r2_description_v2/a_r2_description_v2/urdf/a_r2.xacro (robot description, xacro)
@@ -181,5 +181,5 @@
   <child link="link6_1"/>
   <axis xyz="1.0 0.0 0.0"/>
-  <limit upper="0.0" lower="0.0" effort="100" velocity="100"/>
+  <limit upper="0.1" lower="-0.1" effort="100" velocity="100"/>
 </joint>
 </robot>
